File: sata_connectors.kicad_sch (KiCad schematic)
At the start: 62 parts, among them CN1 HDGCYLSY-SATA-113, CN2 HYCW04-SATA07-129B, Q1 2N7002, Q2 2N7002, Q3 2N7002, Q4 2N7002, Q5 2N7002, U4 TPS259530DSGR, U5 TPS259540DSGR, U6 MCP6002T-I_SN

Commit message: Preliminary revision of USB hub and temperature monitor
Parts:
- U6: value MCP6002T-I_SN -> MCP6002-I_SN; footprint JLCImport:MCP6002T-I_SN -> JLCImport:MCP6002-I_SN; LCSC C7377 -> C116706; Manufacturer Part MCP6002T-I/SN -> MCP6002-I/SN
Other:
- note added: "Source MCP6002 from Microchip's free samples <3"
Changed lines of the file:
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@@
 	(generator_version "10.0")
 	(paper "A4")
+	(text "Source MCP6002 from Microchip's\nfree samples <3"
+		(exclude_from_sim no)
+		(at 111.506 108.204 0)
+		(effects
+			(font
+				(size 0.8128 0.8128)
+				(thickness 0.1588)
+			)
+		)
+	)
 	(text "To ensure compatability with\nDAS/DSS pin, MCU grounds\nDAS/DSS for <x>s on boot"
 		(exclude_from_sim no)
@@
 			)
 		)
-		(property "Value" "MCP6002T-I_SN"
+		(property "Value" "MCP6002-I_SN"
 			(at 111.76 87.63 0)
 			(show_name no)
@@
 			)
 		)
-		(property "Footprint" "JLCImport:MCP6002T-I_SN"
-			(at 111.76 96.52 0)
+		(property "Footprint" "JLCImport:MCP6002-I_SN"
+			(at 111.76 120.904 0)
 			(hide yes)
 			(show_name no)
@@
 			)
 		)
-		(property "Datasheet" "https://www.lcsc.com/datasheet/lcsc_datasheet_2304140030_Microchip-Tech-MCP6002T-I-SN_C7377.pdf"
-			(at 111.76 96.52 0)
+		(property "Datasheet" "https://www.lcsc.com/datasheet/lcsc_datasheet_2412041357_Microchip-Tech-MCP6002-I-SN_C116706.pdf"
+			(at 114.046 126.746 0)
 			(hide yes)
 			(show_name no)
@@
 			)
 		)
-		(property "Description" "-40℃~+125℃ 1.8V~6V 100uA 1MHz 1pA 1pA 2 23mA 28nV/√Hz@1kHz 2uV/℃ 4.5mV 600V/ms 76dB 7V Rail-to-Rail Input, Rail-to-Rail Output SOIC-8 Operational Amplifier ROHS"
-			(at 111.76 96.52 0)
+		(property "Description" "-40℃~+85℃ 1.8V~5.5V 100uA 1MHz 1pA 1pA 2 23mA 28nV/√Hz@1kHz 2uV/℃ 4.5mV 5.5V 600V/ms 76dB Rail-to-Rail Input, Rail-to-Rail Output SOIC-8 Operational Amplifier ROHS"
+			(at 114.046 126.746 0)
 			(hide yes)
 			(show_name no)
@@
 			)
 		)
-		(property "LCSC" "C7377"
-			(at 111.76 96.52 0)
+		(property "LCSC" "C116706"
+			(at 112.014 130.556 0)
 			(hide yes)
 			(show_name no)
@@
 		)
 		(property "Manufacturer" "Microchip Tech"
-			(at 111.76 96.52 0)
+			(at 112.014 124.714 0)
 			(hide yes)
 			(show_name no)
@@
 			)
 		)
-		(property "Manufacturer Part" "MCP6002T-I/SN"
-			(at 111.76 96.52 0)
+		(property "Manufacturer Part" "MCP6002-I/SN"
+			(at 111.506 123.19 0)
 			(hide yes)
 			(show_name no)

Commit message: Preliminary design of power monitor for PSU rails and USB-C VBUS
Connections:
- net PSU_+3V3DC is gone; now on net +3V3: C0.2, CN1.8 (3.3V), CN1.9 (3.3V), R1.2, R4.2
- net PSU_+12V1DC renamed +12V
- net PSU_+5VDC renamed +5V
- no-connect marks 0 -> 1

Commit message: Mostly complete initial transfer to hierarchical schematic
Parts:
- removed ACT_LED1: 0805G_Green, JLCImport:0805G_Green, symbol JLCImport:0805G_Green
- removed C0, C1_0, C1_1: 100nF, Capacitor_SMD:C_0402_1005Metric, symbol JLCImport:CL05B104KB54PNC
- removed C1, C2: 470nF, Capacitor_SMD:C_0603_1608Metric, symbol JLCImport:CL10B474KA8NNNC
- removed C2_0, C2_1, C3, C4: 10uF, Capacitor_SMD:C_0603_1608Metric, symbol JLCImport:CL10A106KP8NNNC
- removed CN1: HDGCYLSY-SATA-113, JLCImport:HDGCYLSY-SATA-113, symbol JLCImport:HDGCYLSY-SATA-113
- removed CN2: HYCW04-SATA07-129B, JLCImport:HYCW04-SATA07-129B, symbol JLCImport:HYCW04-SATA07-129B
- removed CdVdt0, CdVdt1: 22nF, Capacitor_SMD:C_0603_1608Metric, symbol JLCImport:CL10B223KB8NNNC
- removed Cout_0_0, Cout_0_1, Cout_1_0, Cout_1_1, Cout_2_0, Cout_2_1, Cout_3_0, Cout_3_1, Cout_4_0, Cout_4_1: 22uF, Capacitor_SMD:C_1206_3216Metric, symbol JLCImport:CL31A226KAHNNNE
- removed D1: SMAJ13A, Diode_SMD:D_SMA, symbol Diode:SMAJ13A
- removed D2, D5: SS34, Package_DFN_QFN:DHVQFN-20-1EP_2.5x4.5mm_P0.5mm_EP1x3mm, symbol JLCImport:SS34_C8678
- removed D4: SMAJ6.0A, Connector_Hirose_DF40:Hirose_DF40HC(3.5)-20DS-0.4V_2x10_P0.4mm, symbol JLCImport:SMAJ6_0A_C353434
- removed PRES_LED1: whiteLEDSMD, JLCImport:whiteLEDSMD, symbol JLCImport:whiteLEDSMD
- removed Q1, Q2, Q3, Q4, Q5: 2N7002, Package_TO_SOT_SMD:SOT-23-3, symbol JLCImport:2N7002
- removed R1, R23, R24, R25, R28, R4, RFLT0, RFLT1: 10k, Resistor_SMD:R_0402_1005Metric, symbol JLCImport:0402WGF1002TCE
- removed R1_0: 2k, Resistor_SMD:R_0603_1608Metric, symbol JLCImport:0603WAF2001T5E
- removed R1_1: 220k, Resistor_SMD:R_0603_1608Metric, symbol JLCImport:0603WAF220KT5E
- removed R1_2: 68k, Resistor_SMD:R_0603_1608Metric, symbol JLCImport:0603WAF6802T5E
- removed R2, R6: 10, Resistor_SMD:R_0402_1005Metric, symbol JLCImport:0402WGF100JTCE
- removed R22, R8: 120k, Resistor_SMD:R_0603_1608Metric, symbol JLCImport:0603WAF1203T5E
- removed R26, R27: 330, Resistor_SMD:R_0402_1005Metric, symbol JLCImport:0402WGF3300TCE
- removed R2_1, R2_2: 24k, Resistor_SMD:R_0603_1608Metric, symbol JLCImport:0603WAF2402T5E
- removed R3, R5: 300, Resistor_SMD:R_0603_1608Metric, symbol JLCImport:0603WAF3000T5E
- removed R7, R9: 30k, Resistor_SMD:R_0603_1608Metric, symbol JLCImport:0603WAF3002T5E
- removed RILM0: 680, Resistor_SMD:R_0603_1608Metric, symbol JLCImport:0603WAF6800T5E
- removed RILM1: 1k, Resistor_SMD:R_0603_1608Metric, symbol JLCImport:0603WAF1001T5E
- removed U4: TPS259530DSGR, Package_SON:WSON-8-1EP_3x3mm_P0.5mm_EP1.2x2mm, symbol JLCImport:TPS259530DSGR
- removed U5: TPS259540DSGR, Package_SON:WSON-8-1EP_3x3mm_P0.5mm_EP1.2x2mm, symbol JLCImport:TPS259540DSGR
- removed U6: MCP6002-I_SN, JLCImport:MCP6002-I_SN, symbol JLCImport:MCP6002T-I_SN
Connections:
- no-connect marks 1 -> 0
Other:
- note removed: "GPIO pin of MCU controls MOSFET, shorts EN/UVLO to GND when HIGH"
- note removed: "LED Activity Circuit Shows Activity of SATA drive using DAS/DSS pin of SATA Connector"
- note removed: "LED Presence Circuit Shows presence of SATA drive"
- note removed: "Pull down res so MOSFET is closed when GPIO pin is floating (power ON)"
- note removed: "RC filter w/ 48Hz cutoff to prevent HDD noise from affecting HDD power"
- note removed: "Source MCP6002 from Microchip's free samples <3"
- note removed: "To ensure compatability with DAS/DSS pin, MCU grounds DAS/DSS for <x>s on boot"
