File: TC358743.kicad_sch (KiCad schematic)
At the start: 44 parts, among them P1 22P_FPC, U7 TC358743XBG_EL_NOK, U8 TLV62568DBVR, U9 TLV62568DBVR, X2 27MHz

Commit message: Mostly complete initial transfer to hierarchical schematic
Parts:
- removed P1: 22P_FPC, Package_SO:TSSOP-50_4.4x12.5mm_P0.5mm, symbol JLCImport:FPC_0_5MM_22P_Pull_type_H2_0mm_Pick_up
- renumbered C47 to C19, C48 to C20, C5 to C22, C44 to C23, C43 to C27, C42 to C38, C38 to C40, C40 to C42, C7 to C43, C20 to C44, C6 to C45, C22 to C46, C19 to C47, C23 to C48, C49 to C5, C45 to C6, C46 to C7, R35 to R29, R36 to R30, R37 to R31, R38 to R32, R41 to R33, R40 to R34, R39 to R35, R42 to R36, R43 to R37, R31 to R38, R29 to R39, R30 to R40, R33 to R41, R34 to R42, R32 to R43
Connections:
- net HPDI: no longer U7.H2 (HPDI)
- new net HDMI_HPD: U7.H2 (HPDI)
- no-connect marks 6 -> 4

Commit message: Transferred everything to hierarchical schematic and wired PSU power on circuit AND created duplicate schematics for all relevant subsystems
Other:
- moved on the sheet: R39, R40
