File: sensors.kicad_sch (KiCad schematic)
At the start: 11 parts, among them U25 PAC1954T-E_4MX

Commit message: Transferred everything to hierarchical schematic and wired PSU power on circuit AND created duplicate schematics for all relevant subsystems
Parts:
- removed R149, R150: 100k, Resistor_SMD:R_0402_1005Metric, symbol JLCImport:0402WGF1003TCE
- removed R151, R156, R157: 10k, Resistor_SMD:R_0402_1005Metric, symbol JLCImport:0402WGF1002TCE
- removed R152, R153: 510mΩ ±5%, Resistor_SMD:R_1210_3225Metric, symbol JLCImport:YHR1206SE1WR003F5
- removed R154, R155: 180mΩ ±5%, Resistor_SMD:R_0508_1220Metric, symbol JLCImport:LTR10EVHJLR18
- removed R158: 499, Resistor_SMD:R_0402_1005Metric, symbol JLCImport:WR04W1R00FTL
- removed U25: PAC1954T-E_4MX, JLCImport:PAC1954T-E_4MX, symbol JLCImport:PAC1954T-E_4MX
Other:
- note removed: "550mA max sense for LicheeRV Nano +5V"
- note removed: "550mA max sense for touch display +3V3"
- note removed: "Addr: 0010 001"
- note removed: "Power monitor for: PS176, TC358743, LicheeRV Nano, and touch display"
- note removed: "Pull down to disable SLOW sampling"
- note removed: "~196mA max sense for PS176 +3V3"
- note removed: "~196mA max sense for TC358743 +3V3"
