File: FPC_CONN.kicad_sch (KiCad schematic)
At the start: 1 part, among them P1 22P_FPC

Commit message: Cleaned up schematic and replaced TC358743XBG with reverse-engineered LT6911C
Parts:
- P1: footprint Package_SO:TSSOP-50_4.4x12.5mm_P0.5mm -> JLCImport:FPC_0_5MM_22P_Pull_type_H2_0mm_Pick_up
Connections:
- net INT: now reaches P1.17
- no-connect marks 2 -> 1
Changed lines of the file:
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@@
-	)
-	(no_connect
-		(at 80.01 78.74)
 	)
 	(no_connect
@@
 	(wire
 		(pts
+			(xy 78.74 78.74) (xy 80.01 78.74)
+		)
+		(stroke
+			(width 0)
+			(type default)
+		)
+	)
+	(wire
+		(pts
 			(xy 78.74 50.8) (xy 80.01 50.8)
 		)
@@
 		(shape input)
 		(at 78.74 71.12 180)
+		(effects
+			(font
+				(size 1.27 1.27)
+			)
+			(justify right)
+		)
+	)
+	(hierarchical_label "INT"
+		(shape input)
+		(at 78.74 78.74 180)
 		(effects
 			(font
@@
 	)
 	(hierarchical_label "CSI_SCL"
-		(shape input)
+		(shape output)
 		(at 78.74 86.36 180)
 		(effects
@@
 	)
 	(symbol
+		(lib_name "FPC_0_5MM_22P_Pull_type_H2_0mm_Pick_up_1")
 		(lib_id "JLCImport:FPC_0_5MM_22P_Pull_type_H2_0mm_Pick_up")
 		(at 85.09 64.77 0)
@@
 		(in_pos_files yes)
 		(dnp no)
+		(fields_autoplaced yes)
 		(property "Reference" "P1"
-			(at 78.74 94.234 0)
+			(at 93.98 63.4999 0)
 			(show_name no)
 			(do_not_autoplace no)
@@
 		)
 		(property "Value" "22P_FPC"
-			(at 78.74 96.774 0)
+			(at 93.98 66.0399 0)
 			(show_name no)
 			(do_not_autoplace no)
@@
 			)
 		)
-		(property "Footprint" "Package_SO:TSSOP-50_4.4x12.5mm_P0.5mm"
+		(property "Footprint" "JLCImport:FPC_0_5MM_22P_Pull_type_H2_0mm_Pick_up"
 			(at 85.09 64.77 0)
 			(hide yes)
@@
 			)
 		)
+		(pin "8"
+		)
+		(pin "14"
+		)
+		(pin "2"
+		)
+		(pin "1"
+		)
+		(pin "9"
+		)
+		(pin "10"
+		)
+		(pin "13"
+		)
+		(pin "16"
+		)
+		(pin "18"
+		)
+		(pin "5"
+		)
+		(pin "4"
+		)
+		(pin "6"
+		)
+		(pin "3"
+		)
+		(pin "7"
+		)
+		(pin "11"
+		)
+		(pin "12"
+		)
 		(pin "15"
 		)
+		(pin "17"
+		)
+		(pin "19"
+		)
+		(pin "20"
+		)
+		(pin "23"
+		)
 		(pin "22"
 		)
-		(pin "12"
-		)
-		(pin "17"
-		)
-		(pin "16"
-		)
 		(pin "21"
 		)
-		(pin "14"
-		)
-		(pin "23"
-		)
 		(pin "24"
 		)
-		(pin "18"
-		)
-		(pin "13"
-		)
-		(pin "19"
-		)
-		(pin "20"
-		)
-		(pin "8"
-		)
-		(pin "4"
-		)
-		(pin "9"
-		)
-		(pin "10"
-		)
-		(pin "11"
-		)
-		(pin "5"
-		)
-		(pin "6"
-		)
-		(pin "2"
-		)
-		(pin "3"
-		)
-		(pin "1"
-		)
-		(pin "7"
-		)
 		(instances
