File: RTL9210b_0.kicad_sch (KiCad schematic)
At the start: 39 parts, among them CN3 W25Q128FVIQ_Connector, U1 25MHz 10pF, U12 MIC2545A-2YM-TR, U2 RTL9210B-CG, U3 MIC2545A-1YM

Commit message: Added TVS clamping diodes to upstream USB-C port and fixed RX/TX orientation routing for entire system
Parts:
- renumbered C49 to C100, C8 to C19, C9 to C20, C10 to C22, C11 to C23, C12 to C27, C13 to C38, C14 to C39, C15 to C40, C16 to C41, C17 to C42, C18 to C44, C21 to C46, C24 to C93, C25 to C94, C33 to C95, C34 to C96, C35 to C97, C36 to C98, C37 to C99, CN3 to CN7, L7 to L10, L5 to L8, L6 to L9, R10 to R31, R11 to R32, R12 to R33, R13 to R34, R14 to R35, R15 to R36, R16 to R37, R17 to R38, R18 to R39, R19 to R41, R56 to R58, U12 to U14, U1 to U7, U2 to U8, U3 to U9
