File: MCP6002.kicad_sch (KiCad schematic)
At the start: 9 parts, among them U6 MCP6002-I_SN

Commit message: Changed USB7206C's buck converter to LX7167
Parts:
- removed R22, R8: 120k, Resistor_SMD:R_0603_1608Metric, symbol JLCImport:0603WAF1203T5E
- added R224, R68: 120k, Resistor_SMD:R_0402_1005Metric, symbol JLCImport:HRC0402F1203DNTO
Connections:
- net at R24.1: now also R68.2
- net at R7.2, U6.2 (-INA): now also R68.1
- net at R9.2, U6.6 (-INB): now also R224.1
- net at R23.2: now also R224.2
