File: UCS2113.kicad_sch (KiCad schematic)
At the start: 9 parts, among them U30 UCS2113-1-V_G4

Commit message: Basic Function Review/Documentation of USB7205C
Connections:
- net P6_USB2.0_ALERT# renamed P4_USB2.0_ALERT#
- net P6_USB2.0_VCC renamed P4_USB2.0_VCC
- net PRT_CTL6 renamed PRT_CTL4
Changed lines of the file:
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@@
 		)
 	)
-	(hierarchical_label "PRT_CTL6"
-		(shape input)
+	(hierarchical_label "PRT_CTL4"
+		(shape output)
 		(at 121.92 68.58 0)
 		(effects
@@
 		)
 	)
-	(hierarchical_label "P6_USB2.0_VCC"
+	(hierarchical_label "P4_USB2.0_VCC"
 		(shape output)
 		(at 120.65 77.47 0)
@@
 	)
 	(hierarchical_label "PRT_CTL5"
-		(shape input)
+		(shape output)
 		(at 85.09 55.88 180)
 		(effects
@@
 		)
 	)
-	(hierarchical_label "P6_USB2.0_ALERT#"
+	(hierarchical_label "P4_USB2.0_ALERT#"
 		(shape output)
 		(at 146.05 66.04 0)
