File: PORT5_USB.kicad_sch (KiCad schematic)
At the start: 4 parts

Commit message: Added an (optional) RC network between shield pins of USB connector and GND
Parts:
- renumbered USB4 to USB5
Changed lines of the file:
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@@
 		(dnp no)
 		(fields_autoplaced yes)
-		(property "Reference" "USB4"
+		(property "Reference" "USB5"
 			(at 100.33 52.07 0)
 			(show_name no)
@@
 			(project "serverv2_backplane"
 				(path "/d38d6818-cf53-410d-afa3-a75a85b7c05a/ed95f4dd-0500-4b68-8234-f3e0f9cd2ae3"
-					(reference "USB4")
+					(reference "USB5")
 					(unit 1)
 				)
