File: RP2354B_0.kicad_sch (KiCad schematic)
At the start: 29 parts, among them CN4 W25Q128FVIQ_Connector, J6 Conn_01x02, X3 12MHz

Commit message: Basic Function Review/Documentation of RP2354B
Parts:
- removed BOOTSEL1, RESET1: TS-1088-AR02016, JLCImport:TS-1088-AR02016, symbol JLCImport:TS-1088-AR02016
- removed C51: 4.7uF, Capacitor_SMD:C_0402_1005Metric, symbol JLCImport:CL05A475MP5NRNC
- removed C65, C66: 33pF, Capacitor_SMD:C_0402_1005Metric, symbol JLCImport:0402CG330J500NT
- removed CN4: W25Q128FVIQ_Connector, JLCImport:H2541FV-C762-2X04P, symbol JLCImport:H2541FV-C762-2X04P
- removed J6: Conn_01x02, Connector_PinHeader_2.54mm:PinHeader_1x02_P2.54mm_Vertical, symbol Connector_Generic:Conn_01x02
- removed L4: 3.3uH, JLCImport:AOTA-B201610S3R3-101-T, symbol JLCImport:AOTA-B201610S3R3-101-T
- removed R48: 1k, Resistor_SMD:R_0402_1005Metric, symbol JLCImport:0402WGF1001TCE
- removed R49: 220, Resistor_SMD:R_0603_1608Metric, symbol JLCImport:0603WAF2200T5E
- removed X3: 12MHz, JLCImport:X322512MSB4SI, symbol JLCImport:X322512MSB4SI
- added C263: 4.7uF, Capacitor_SMD:C_0402_1005Metric, symbol JLCImport:CL05A475MP5NRNC
- added C51, C81: 15pF, Capacitor_SMD:C_0402_1005Metric, symbol JLCImport:0402CG150J500NT
- added C75, C78: 100nF, Capacitor_SMD:C_0402_1005Metric, symbol JLCImport:CL05B104KB54PNC
- added CRYSTAL1: CM4012M00010001, Crystal:Crystal_SMD_2520-4Pin_2.5x2.0mm, symbol JLCImport:CM4012M00010001
- added L2: 3.3uH, JLCImport:PIM252010S3R3MBCA, symbol JLCImport:PIM252010S3R3MBCA
- added R191, R51, R55: 10k, Resistor_SMD:R_0402_1005Metric, symbol JLCImport:0402WGF1002TCE
- added TP1, TP4: UART TX Pad, TestPoint:TestPoint_Pad_2.0x2.0mm, symbol Connector:TestPoint
- added TP7: Reset pad, TestPoint:TestPoint_Pad_2.0x2.0mm, symbol Connector:TestPoint
- PI1: LCSC (none) -> C39843328
Connections:
- net +1V1: now also C263.1, C78.2, L2.2
- net +3V3: now also C75.2, R191.2, R51.2, R55.2
- net GND: now also C263.2, C51.1, C75.1, C78.1, C81.1, CRYSTAL1.2 (GND), CRYSTAL1.4 (GND)
- net IRQ1: now also R191.1
- net SCL1: now also R55.1; no longer PI1.39 (GPIO31)
- net SDA1: now also R51.1; no longer PI1.38 (GPIO30)
- net XIN: now also C81.2, CRYSTAL1.1
- net XOUT: now also R47.2
- net at PI1.35 (RUN): now also TP7.1
- net at PI1.36 (GPIO28): now also TP1.1
- net at PI1.37 (GPIO29): now also TP4.1
- net at PI1.63 (VREG_LX): now also L2.1
- net at R47.1: now also C51.2, CRYSTAL1.3
- net QSPI_SCLK: no longer names the net of PI1.71 (QSPI_SCLK)
- net QSPI_SD0: no longer names the net of PI1.72 (QSPI_SD0)
- net QSPI_SD1: no longer names the net of PI1.74 (QSPI_SD1)
- net QSPI_SD2: no longer names the net of PI1.73 (QSPI_SD2)
- net QSPI_SD3: no longer names the net of PI1.70 (QSPI_SD3)
- net QSPI_SS: no longer names the net of PI1.75 (~{QSPI_SS})
- net QSPI_SS: no longer R47.2
- no-connect marks 6 -> 14
Other:
- note added: "UART debug pads"
- note removed: "Dual 33pF capacitors is to achieve 16.5pF + ~3pF (parasitic) = ~19.5pF total, but 220ohm res is eyeballed, needs testing"
- note removed: "I2C, to slave devices"
- note removed: "Reset Button"
- note removed: "There's a lot of extra resistors on CS# in the example design, but they label them as DNF, so I've excluded them."
- note removed: "UART debug pins"
- note removed: "USB Boot Button Default -> Flash boot"
