File: SG2002_HEADER.kicad_sch (KiCad schematic)
At the start: 2 parts, among them J2 Conn_01x14, J3 Conn_01x14

Commit message: Transferred everything to hierarchical schematic and wired PSU power on circuit AND created duplicate schematics for all relevant subsystems
Connections:
- net +3V3: no longer names the net of J3.3V3 (Pin_1)
- net SCL0 renamed SCL1
- net SDA0 renamed SDA1
- no-connect marks 7 -> 8
Changed lines of the file:
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@@
+	)
+	(no_connect
+		(at 109.22 77.47)
 	)
 	(no_connect
@@
 	(wire
 		(pts
-			(xy 106.68 78.74) (xy 106.68 77.47)
-		)
-		(stroke
-			(width 0)
-			(type default)
-		)
-	)
-	(wire
-		(pts
 			(xy 62.23 59.69) (xy 86.36 59.69)
 		)
@@
 	(wire
 		(pts
+			(xy 109.22 77.47) (xy 106.68 77.47)
+		)
+		(stroke
+			(width 0)
+			(type default)
+		)
+	)
+	(wire
+		(pts
 			(xy 62.23 52.07) (xy 86.36 52.07)
 		)
@@
 	(wire
 		(pts
-			(xy 106.68 78.74) (xy 114.3 78.74)
-		)
-		(stroke
-			(width 0)
-			(type default)
-		)
-	)
-	(wire
-		(pts
 			(xy 62.23 72.39) (xy 86.36 72.39)
 		)
@@
 		(shape input)
 		(at 149.86 74.93 0)
-		(effects
-			(font
-				(size 1.27 1.27)
-			)
-			(justify left)
-		)
-	)
-	(hierarchical_label "+3V3"
-		(shape input)
-		(at 114.3 78.74 0)
 		(effects
 			(font
@@
 			(font
 				(size 1.27 1.27)
+				(color 53 217 18 1)
 			)
 			(justify left)
@@
 		)
 	)
-	(hierarchical_label "SCL0"
+	(hierarchical_label "SCL1"
 		(shape output)
 		(at 152.4 59.69 0)
@@
 			(font
 				(size 1.27 1.27)
+				(color 220 155 18 1)
 			)
 			(justify left)
@@
 		)
 	)
-	(hierarchical_label "SDA0"
+	(hierarchical_label "SDA1"
 		(shape bidirectional)
 		(at 152.4 64.77 0)
@@
 			(font
 				(size 1.27 1.27)
+				(color 220 155 18 1)
 			)
 			(justify left)
@@
 			(font
 				(size 1.27 1.27)
+				(color 53 217 18 1)
 			)
 			(justify left)
@@
 		)
 	)
-	(symbol
-		(lib_id "power:+5V")
-		(at 114.3 78.74 0)
-		(unit 1)
-		(body_style 1)
-		(exclude_from_sim no)
-		(in_bom yes)
-		(on_board yes)
-		(in_pos_files yes)
-		(dnp no)
-		(property "Reference" "#PWR0116"
-			(at 114.3 82.55 0)
-			(hide yes)
-			(show_name no)
-			(do_not_autoplace no)
-			(effects
-				(font
-					(size 1.27 1.27)
-				)
-			)
-		)
-		(property "Value" "+3V3"
-			(at 110.49 77.47 0)
-			(show_name no)
-			(do_not_autoplace no)
-			(effects
-				(font
-					(size 1.27 1.27)
-				)
-			)
-		)
-		(property "Footprint" ""
-			(at 114.3 78.74 0)
-			(hide yes)
-			(show_name no)
-			(do_not_autoplace no)
-			(effects
-				(font
-					(size 1.27 1.27)
-				)
-			)
-		)
-		(property "Datasheet" ""
-			(at 114.3 78.74 0)
-			(hide yes)
-			(show_name no)
-			(do_not_autoplace no)
-			(effects
-				(font
-					(size 1.27 1.27)
-				)
-			)
-		)
-		(property "Description" "Power symbol creates a global label with name \"+5V\""
-			(at 114.3 78.74 0)
-			(hide yes)
-			(show_name no)
-			(do_not_autoplace no)
-			(effects
-				(font
-					(size 1.27 1.27)
-				)
-			)
-		)
-		(pin "1"
-		)
-		(instances
-			(project "serverv2_backplane"
-				(path "/d38d6818-cf53-410d-afa3-a75a85b7c05a/d5a67228-81b6-43a9-8d9d-64c8ba4d62b6"
-					(reference "#PWR0116")
-					(unit 1)
-				)
-			)
-		)
-	)

Commit message: Basic Function Review/Documentation of RP2354B
Parts:
- added R189, R190: 10k, Resistor_SMD:R_0402_1005Metric, symbol JLCImport:0402WGF1002TCE
Connections:
- net SCL1: now also R189.1
- net SDA1: now also R190.1
- new net +3V3: R189.2, R190.2
