File: TPS65987D.kicad_sch (KiCad schematic)
At the start: 16 parts, among them CN5 W25Q128FVIQ_Connector, U15 TPS65987DDHRSHR

Commit message: Basic Function Review/Documentation of RP2354B
Parts:
- removed CN5: W25Q128FVIQ_Connector, JLCImport:H2541FV-C762-2X04P, symbol JLCImport:H2541FV-C762-2X04P
- removed R72: 24k, Resistor_SMD:R_0603_1608Metric, symbol JLCImport:0603WAF2402T5E
- removed R73: 75k, Resistor_SMD:R_0603_1608Metric, symbol JLCImport:0603WAF7502T5E
- removed R75, R76, R77, R78: 3.3k, Resistor_SMD:R_0402_1005Metric, symbol JLCImport:0402WGF3301TCE
- removed U15: TPS65987DDHRSHR, Package_DFN_QFN:VQFN-40-1EP_5x5mm_P0.4mm_EP3.3x3.3mm, symbol JLCImport:TPS65987DDHRSHR
- added C210: 4.7uF, Capacitor_SMD:C_0603_1608Metric, symbol JLCImport:CL10A475KL8NRNC
- added R72: 20k, Resistor_SMD:R_0402_1005Metric, symbol JLCImport:1RC0402J0203
- added R73: 120k, Resistor_SMD:R_0402_1005Metric, symbol JLCImport:HRC0402F1203DNTO
- added R75: 100k, Resistor_SMD:R_0402_1005Metric, symbol JLCImport:0402WGF1003TCE
- added U13: TPS65987DDHRSHR, JLCImport:TPS65987DDHRSHR, symbol JLCImport:TPS65987DDHRSHR
Connections:
- net +3V3: now also U13.5 (VIN_3V3)
- net +5V: now also U13.25 (PP_CABLE)
- net CC1: now also U13.24 (C_CC1)
- net CC2: now also U13.26 (C_CC2)
- net CTRL_IRQ2: now also U13.34 (I2C2_IRQ)
- net CTRL_SCL1: now also U13.27 (I2C1_SCL)
- net CTRL_SCL2: now also U13.32 (I2C2_SCL)
- net CTRL_SCL3: now also U13.21 (I2C3_SCL(GPIO5))
- net CTRL_SDA1: now also U13.28 (I2C1_SDA)
- net CTRL_SDA2: now also U13.33 (I2C2_SDA)
- net CTRL_SDA3: now also U13.22 (I2C3_SDA(GPIO6))
- net DP_HPD: now also U13.30 (HPD(GPIO3))
- net DRAIN1: now also U13.15 (DRAIN1), U13.19 (DRAIN1), U13.58 (DRAIN1), U13.8 (DRAIN1)
- net DRAIN2: now also U13.52 (DRAIN2), U13.56 (DRAIN2), U13.57 (DRAIN2), U13.7 (DRAIN2)
- net GND: now also C210.2, R72.1, R75.1, U13.20 (GND), U13.36 (SPI_PICO(GPIO8)), U13.37 (SPI_POCI(GPIO9)), U13.38 (SPI_CLK(GPIO10)), U13.39 (SPI_CS(GPIO11)), U13.45 (GND), U13.46 (GND), U13.47 (GND), U13.51 (GND), U13.59 (GND)
- net PP_HV: now also U13.1 (PP_HV2), U13.11 (PP_HV1), U13.12 (PP_HV1), U13.2 (PP_HV2)
- net VBUS: now also U13.13 (VBUS1), U13.14 (VBUS1), U13.3 (VBUS2), U13.4 (VBUS2)
- net at R74.1: now also U13.44 (HRESET)
- net CTRL_LDO_3V3 renamed LDO_3V3
- net LDO_3V3: now also R73.2, U13.9 (LDO_3V3)
- new net: R75.2, U13.10 (ADCIN2)
- new net: R72.2, R73.1, U13.6 (ADCIN1)
- new net LDO_1V8: C210.1, U13.35 (LDO_1V8)
Other:
- note added: "SPI_POCI=0 + DIV=0.14 for BP_NoResponse + Config 2"
- note removed: "SPI_POCI=0 + DIV=0.24 for BP_NoWait + conf 2"

Commit message: Basic Function Review/Documentation for TPS65987D
Parts:
- removed C112, C26: 10uF, Capacitor_SMD:C_0603_1608Metric, symbol JLCImport:CL10A106KP8NNNC
- removed C113, C114: 10uF, Capacitor_SMD:C_0805_2012Metric, symbol JLCImport:CL21A106KAYNNNE
- added C113, C211, C212, C236: 10uF, Capacitor_SMD:C_0603_1608Metric, symbol JLCImport:HGC0603R5106M350NTHJ
Connections:
- net +3V3: now also C212.2
- net GND: now also C113.1, C211.1, C212.1, C236.1
- net LDO_3V3: now also C211.2
- net PP_HV: now also C113.2, C236.2
Other:
- note removed: "BC1.2 not used so leave C_USB floating - verify this"
