File: TPS55288.kicad_sch (KiCad schematic)
At the start: 34 parts, among them Q6 CSD18513Q5A, Q7 CSD18513Q5A, U10 TPS55288RPMR

Commit message: TPS55288: Added extra 220uF bypass capacitor on VOUT and connected SW1/SW2 properly
Parts:
- removed C115, C116, C117, C118: 10uF, Capacitor_SMD:C_0805_2012Metric, symbol JLCImport:CL21A106KAYNNNE
- removed L12: 4.7uH, JLCImport:SL1040-4R7M, symbol JLCImport:SL1040-4R7M
- removed R84: 6.2k, Resistor_SMD:R_0603_1608Metric, symbol JLCImport:0603WAF6201T5E
- added C112, C114, C115, C116: 10uF, Capacitor_SMD:C_0603_1608Metric, symbol JLCImport:TCC0603X5R106K250CT
- added C132: 1uF, Capacitor_SMD:C_0402_1005Metric, symbol JLCImport:CL05A105KA5NQNC
- added C26: 220uF, JLCImport:RVT1V221M0810-C72498, symbol JLCImport:RVT1V221M0810-C72498
- added L12: 4.7uF, JLCImport:XR1265-4R7M, symbol JLCImport:XR1265-4R7M
Connections:
- net AGND: now also C112.1, C114.1, C115.1, C116.1, C132.1, C26.2
- net ISP: now also C112.2, C114.2, C115.2, C116.2, C26.1
- net PP_HV: now also C132.2
- net SW2: now also L12.2
- net SW1: now reaches Q6.5 (D), Q6.6 (D), Q6.7 (D), Q6.8 (D), Q6.9 (D), Q7.1 (S), Q7.2 (S), Q7.3 (S)
- net SW1: now also C120.2, U10.23 (SW1), L12.1
- no-connect marks 0 -> 1
Other:
- note added: "Float MODE to set PFM"
- note added: "High-side power MOSFET"
- note added: "Low-side power MOSFET"
- note removed: "6.2k b/w MODE and GND to set I2C addr, per EVM"
- note removed: "This inductor does not meet the recommended DCR spec; hopefully it still works!!"
- moved on the sheet: C119, C120, C121, C122, C123, C124, C125, C126, C127, C128, C129, C130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
