File: serverv2_backplane.kicad_sch (KiCad schematic)
At the start: 0 parts

Commit message: Basic Function Review/Documentation of RP2354B
Other:
- sheet RP2350B_0 renamed RP2354B_0
- sheet RP2350B_1 renamed RP2354B_1
- sheet RP2350B_2 renamed RP2354B_2
- sheet RP2354B_0: file RP2350B_0.kicad_sch -> RP2354B_0.kicad_sch
- sheet RP2354B_1: file RP2350B_0.kicad_sch -> RP2354B_0.kicad_sch
- sheet RP2354B_2: file RP2350B_0.kicad_sch -> RP2354B_0.kicad_sch
- sheet SG2002_HEADER ports: added +3V3; removed none
Changed lines of the file:
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@@
 	(wire
 		(pts
-			(xy 92.71 213.36) (xy 88.9 213.36)
+			(xy 92.71 213.36) (xy 87.63 213.36)
 		)
 		(stroke
@@
 	(wire
 		(pts
-			(xy 88.9 213.36) (xy 88.9 232.41)
+			(xy 87.63 213.36) (xy 87.63 232.41)
 		)
 		(stroke
@@
 	(wire
 		(pts
+			(xy 236.22 193.04) (xy 240.03 193.04)
+		)
+		(stroke
+			(width 0)
+			(type default)
+		)
+	)
+	(wire
+		(pts
 			(xy 237.49 240.03) (xy 240.03 240.03)
 		)
@@
 	(wire
 		(pts
-			(xy 88.9 232.41) (xy 92.71 232.41)
+			(xy 87.63 232.41) (xy 92.71 232.41)
 		)
 		(stroke
@@
 	)
 	(global_label "USB7205C_SCL"
-		(shape input)
+		(shape output)
 		(at 276.86 227.33 180)
 		(fields_autoplaced yes)
@@
 	)
 	(symbol
+		(lib_id "power:+5V")
+		(at 236.22 193.04 0)
+		(unit 1)
+		(body_style 1)
+		(exclude_from_sim no)
+		(in_bom yes)
+		(on_board yes)
+		(in_pos_files yes)
+		(dnp no)
+		(property "Reference" "#PWR0641"
+			(at 236.22 196.85 0)
+			(hide yes)
+			(show_name no)
+			(do_not_autoplace no)
+			(effects
+				(font
+					(size 1.27 1.27)
+				)
+			)
+		)
+		(property "Value" "+3V3"
+			(at 236.22 188.722 0)
+			(show_name no)
+			(do_not_autoplace no)
+			(effects
+				(font
+					(size 1.27 1.27)
+				)
+			)
+		)
+		(property "Footprint" ""
+			(at 236.22 193.04 0)
+			(hide yes)
+			(show_name no)
+			(do_not_autoplace no)
+			(effects
+				(font
+					(size 1.27 1.27)
+				)
+			)
+		)
+		(property "Datasheet" ""
+			(at 236.22 193.04 0)
+			(hide yes)
+			(show_name no)
+			(do_not_autoplace no)
+			(effects
+				(font
+					(size 1.27 1.27)
+				)
+			)
+		)
+		(property "Description" "Power symbol creates a global label with name \"+5V\""
+			(at 236.22 193.04 0)
+			(hide yes)
+			(show_name no)
+			(do_not_autoplace no)
+			(effects
+				(font
+					(size 1.27 1.27)
+				)
+			)
+		)
+		(pin "1"
+		)
+		(instances
+			(project "serverv2_backplane"
+				(path "/d38d6818-cf53-410d-afa3-a75a85b7c05a"
+					(reference "#PWR0641")
+					(unit 1)
+				)
+			)
+		)
+	)
+	(symbol
 		(lib_id "power:GND")
 		(at 393.7 391.16 0)
@@
 			(color 0 0 0 0)
 		)
-		(property "Sheetname" "RP2350B_1"
+		(property "Sheetname" "RP2354B_1"
 			(at 278.13 185.9784 0)
 			(show_name no)
@@
 			)
 		)
-		(property "Sheetfile" "RP2350B_0.kicad_sch"
+		(property "Sheetfile" "RP2354B_0.kicad_sch"
 			(at 278.13 310.4646 0)
 			(hide yes)
@@
 			(color 0 0 0 0)
 		)
-		(property "Sheetname" "RP2350B_0"
+		(property "Sheetname" "RP2354B_0"
 			(at 200.66 19.6084 0)
 			(show_name no)
@@
 			)
 		)
-		(property "Sheetfile" "RP2350B_0.kicad_sch"
+		(property "Sheetfile" "RP2354B_0.kicad_sch"
 			(at 200.66 109.1696 0)
 			(hide yes)
@@
 			(color 0 0 0 0)
 		)
-		(property "Sheetname" "RP2350B_2"
+		(property "Sheetname" "RP2354B_2"
 			(at 278.13 326.9484 0)
 			(show_name no)
@@
 			)
 		)
-		(property "Sheetfile" "RP2350B_0.kicad_sch"
+		(property "Sheetfile" "RP2354B_0.kicad_sch"
 			(at 278.13 431.1146 0)
 			(hide yes)
@@
 			(effects
 				(font
+					(size 1.27 1.27)
+				)
+				(justify left)
+			)
+		)
+		(pin "+3V3" input
+			(at 240.03 193.04 180)
+			(effects
+				(font

Commit message: Basic Function Review/Documentation for TPS65987D
Changed lines of the file:
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@@
 	(wire
 		(pts
-			(xy 81.28 106.68) (xy 90.17 106.68)
+			(xy 81.28 101.6) (xy 90.17 101.6)
 		)
 		(stroke
@@
 	(wire
 		(pts
-			(xy 107.95 110.49) (xy 107.95 118.11)
-		)
-		(stroke
-			(width 0)
-			(type default)
-		)
-	)
-	(wire
-		(pts
 			(xy 182.88 420.37) (xy 199.39 420.37)
 		)
@@
 	(wire
 		(pts
-			(xy 81.28 237.49) (xy 92.71 237.49)
-		)
-		(stroke
-			(width 0)
-			(type default)
-		)
-	)
-	(wire
-		(pts
 			(xy 316.23 368.3) (xy 356.87 368.3)
 		)
@@
 	(wire
 		(pts
-			(xy 81.28 106.68) (xy 81.28 237.49)
+			(xy 81.28 101.6) (xy 81.28 237.49)
 		)
 		(stroke
@@
 	(wire
 		(pts
+			(xy 107.95 110.49) (xy 107.95 118.11)
+		)
+		(stroke
+			(width 0)
+			(type default)
+		)
+	)
+	(wire
+		(pts
 			(xy 274.32 190.5) (xy 278.13 190.5)
 		)
@@
 	(wire
 		(pts
+			(xy 81.28 237.49) (xy 92.71 237.49)
+		)
+		(stroke
+			(width 0)
+			(type default)
+		)
+	)
+	(wire
+		(pts
 			(xy 316.23 280.67) (xy 356.87 280.67)
 		)
@@
 			)
 		)
-		(pin "PP_HV" input
-			(at 107.95 118.11 90)
+		(pin "GND" input
+			(at 138.43 146.05 0)
 			(effects
 				(font
@@
 			)
 		)
-		(pin "GND" input
-			(at 138.43 146.05 0)
+		(pin "PP_HV" output
+			(at 107.95 118.11 90)
 			(effects
 				(font
@@
 		)
 		(pin "DP_HPD" input
-			(at 90.17 106.68 180)
+			(at 90.17 101.6 180)
 			(effects
 				(font

Commit message: TPS55288: Added extra 220uF bypass capacitor on VOUT and connected SW1/SW2 properly
Other:
- sheet TPS55288 ports: added +3V3, +5V; removed none
Changed lines of the file:
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@@
 	(wire
 		(pts
+			(xy 138.43 127) (xy 152.4 127)
+		)
+		(stroke
+			(width 0)
+			(type default)
+		)
+	)
+	(wire
+		(pts
 			(xy 389.255 417.83) (xy 393.7 417.83)
 		)
@@
 	(wire
 		(pts
+			(xy 138.43 124.46) (xy 146.05 124.46)
+		)
+		(stroke
+			(width 0)
+			(type default)
+		)
+	)
+	(wire
+		(pts
 			(xy 389.255 386.08) (xy 398.78 386.08)
 		)
@@
 	(symbol
 		(lib_id "power:+5V")
+		(at 146.05 124.46 0)
+		(unit 1)
+		(body_style 1)
+		(exclude_from_sim no)
+		(in_bom yes)
+		(on_board yes)
+		(in_pos_files yes)
+		(dnp no)
+		(fields_autoplaced yes)
+		(property "Reference" "#PWR07"
+			(at 146.05 128.27 0)
+			(hide yes)
+			(show_name no)
+			(do_not_autoplace no)
+			(effects
+				(font
+					(size 1.27 1.27)
+				)
+			)
+		)
+		(property "Value" "+5V"
+			(at 146.05 119.38 0)
+			(show_name no)
+			(do_not_autoplace no)
+			(effects
+				(font
+					(size 1.27 1.27)
+				)
+			)
+		)
+		(property "Footprint" ""
+			(at 146.05 124.46 0)
+			(hide yes)
+			(show_name no)
+			(do_not_autoplace no)
+			(effects
+				(font
+					(size 1.27 1.27)
+				)
+			)
+		)
+		(property "Datasheet" ""
+			(at 146.05 124.46 0)
+			(hide yes)
+			(show_name no)
+			(do_not_autoplace no)
+			(effects
+				(font
+					(size 1.27 1.27)
+				)
+			)
+		)
+		(property "Description" "Power symbol creates a global label with name \"+5V\""
+			(at 146.05 124.46 0)
+			(hide yes)
+			(show_name no)
+			(do_not_autoplace no)
+			(effects
+				(font
+					(size 1.27 1.27)
+				)
+			)
+		)
+		(pin "1"
+		)
+		(instances
+			(project "serverv2_backplane"
+				(path "/d38d6818-cf53-410d-afa3-a75a85b7c05a"
+					(reference "#PWR07")
+					(unit 1)
+				)
+			)
+		)
+	)
+	(symbol
+		(lib_id "power:+5V")
 		(at 398.78 292.1 0)
 		(unit 1)
@@
 	(symbol
 		(lib_id "power:+5V")
+		(at 152.4 127 0)
+		(unit 1)
+		(body_style 1)
+		(exclude_from_sim no)
+		(in_bom yes)
+		(on_board yes)
+		(in_pos_files yes)
+		(dnp no)
+		(fields_autoplaced yes)
+		(property "Reference" "#PWR025"
+			(at 152.4 130.81 0)
+			(hide yes)
+			(show_name no)
+			(do_not_autoplace no)
+			(effects
+				(font
+					(size 1.27 1.27)
+				)
+			)
+		)
+		(property "Value" "+3V3"
+			(at 152.4 121.92 0)
+			(show_name no)
+			(do_not_autoplace no)
+			(effects
+				(font
+					(size 1.27 1.27)
+				)
+			)
+		)
+		(property "Footprint" ""
+			(at 152.4 127 0)
+			(hide yes)
+			(show_name no)
+			(do_not_autoplace no)
+			(effects
+				(font
+					(size 1.27 1.27)
+				)
+			)
+		)
+		(property "Datasheet" ""
+			(at 152.4 127 0)
+			(hide yes)
+			(show_name no)
+			(do_not_autoplace no)
+			(effects
+				(font
+					(size 1.27 1.27)
+				)
+			)
+		)
+		(property "Description" "Power symbol creates a global label with name \"+5V\""
+			(at 152.4 127 0)
+			(hide yes)
+			(show_name no)
+			(do_not_autoplace no)
+			(effects
+				(font
+					(size 1.27 1.27)
+				)
+			)
+		)
+		(pin "1"
+		)
+		(instances
+			(project "serverv2_backplane"
+				(path "/d38d6818-cf53-410d-afa3-a75a85b7c05a"
+					(reference "#PWR025")
+					(unit 1)
+				)
+			)
+		)
+	)
+	(symbol
+		(lib_id "power:+5V")
 		(at 393.7 262.89 0)
 		(unit 1)
@@
 			(effects
 				(font
+					(size 1.27 1.27)
+				)
+				(justify right)
+			)
+		)
+		(pin "+5V" input
+			(at 138.43 124.46 0)
+			(effects
+				(font
+					(size 1.27 1.27)
+				)
+				(justify right)
+			)
+		)
+		(pin "+3V3" input
+			(at 138.43 127 0)
+			(effects
+				(font
