File: pcb_files/SG2002_HEADER.kicad_sch (KiCad schematic)
At the start: 4 parts, among them J2 Conn_01x14, J3 Conn_01x14

Commit message: Changed TPS55288 to internal droop compensation and added current monitoring for TPS55288 to ADC pin of LicheeRV Nano
Connections:
- net ADC: now reaches J3.ADC (Pin_10)
- no-connect marks 8 -> 7
Changed lines of the file:
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@@
 		(at 62.23 62.23)
 	)
-	(no_connect
-		(at 134.62 54.61)
-	)
 	(wire
 		(pts
@@
 	(wire
 		(pts
-			(xy 106.68 54.61) (xy 134.62 54.61)
+			(xy 149.86 74.93) (xy 106.68 74.93)
+		)
+		(stroke
+			(width 0)
+			(type default)
+		)
+	)
+	(wire
+		(pts
+			(xy 43.18 88.9) (xy 55.88 88.9)
+		)
+		(stroke
+			(width 0)
+			(type default)
+		)
+	)
+	(wire
+		(pts
+			(xy 106.68 44.45) (xy 152.4 44.45)
+		)
+		(stroke
+			(width 0)
+			(type default)
+		)
+	)
+	(wire
+		(pts
+			(xy 43.18 99.06) (xy 43.18 101.6)
+		)
+		(stroke
+			(width 0)
+			(type default)
+		)
+	)
+	(wire
+		(pts
+			(xy 152.4 59.69) (xy 106.68 59.69)
+		)
+		(stroke
+			(width 0)
+			(type default)
+			(color 1 167 194 1)
+		)
+	)
+	(wire
+		(pts
+			(xy 43.18 101.6) (xy 58.42 101.6)
+		)
+		(stroke
+			(width 0)
+			(type default)
+		)
+	)
+	(wire
+		(pts
+			(xy 106.68 54.61) (xy 152.4 54.61)
 		)
 		(stroke
@@
 			(type default)
 			(color 118 114 117 1)
-		)
-	)
-	(wire
-		(pts
-			(xy 149.86 74.93) (xy 106.68 74.93)
-		)
-		(stroke
-			(width 0)
-			(type default)
-		)
-	)
-	(wire
-		(pts
-			(xy 43.18 88.9) (xy 55.88 88.9)
-		)
-		(stroke
-			(width 0)
-			(type default)
-		)
-	)
-	(wire
-		(pts
-			(xy 106.68 44.45) (xy 152.4 44.45)
-		)
-		(stroke
-			(width 0)
-			(type default)
-		)
-	)
-	(wire
-		(pts
-			(xy 43.18 99.06) (xy 43.18 101.6)
-		)
-		(stroke
-			(width 0)
-			(type default)
-		)
-	)
-	(wire
-		(pts
-			(xy 152.4 59.69) (xy 106.68 59.69)
-		)
-		(stroke
-			(width 0)
-			(type default)
-			(color 1 167 194 1)
-		)
-	)
-	(wire
-		(pts
-			(xy 43.18 101.6) (xy 58.42 101.6)
-		)
-		(stroke
-			(width 0)
-			(type default)
 		)
 	)
@@
 		)
 	)
+	(hierarchical_label "ADC"
+		(shape input)
+		(at 152.4 54.61 0)
+		(effects
+			(font
+				(size 1.27 1.27)
+				(color 118 114 117 1)
+			)
+			(justify left)
+		)
+	)
