File: pcb_files/PAC1954_FANS.kicad_sch (KiCad schematic)
At the start: 11 parts, among them U27 PAC1954T-E_4MX

Commit message: Basic Function Review/Documentation for MCP9808
Parts:
- removed R170, R171: 100k, Resistor_SMD:R_0402_1005Metric, symbol JLCImport:0402WGF1003TCE
- added R84, R88: 49.9k, Resistor_SMD:R_0402_1005Metric, symbol JLCImport:RMS04FT4992
Connections:
- net +3V3: now also R84.1, R88.2
- net SCL: now also R84.2
- net SDA: now also R88.1

Commit message: Switched PAC1954 to SLOW mode to save power
Parts:
- removed R173: 1.27k, Resistor_SMD:R_0402_1005Metric, symbol JLCImport:WR04X1271FTL
- removed R175: 10k, Resistor_SMD:R_0402_1005Metric, symbol JLCImport:0402WGF1002TCE
- added C250: 100nF, Capacitor_SMD:C_0402_1005Metric, symbol JLCImport:CL05B104KB54PNC
- added C252: 4.7uF, Capacitor_SMD:C_0402_1005Metric, symbol JLCImport:CL05A475MP5NRNC
- added R149: 10k, Resistor_SMD:R_0402_1005Metric, symbol JLCImport:0402WGF1002TCE
Connections:
- net +3V3: now also U27.6 (ADDRSEL), C250.2, C252.2, R149.2
- net GND: now also C250.1, C252.1
- net at U27.1 (SLOW/ALERT1#): now also R149.1
Other:
- note added: "Pull up to enable SLOW sampling"
- note removed: "Pull down to disable SLOW sampling"

Commit message: Added FAN4 and updated RP2354/PAC1954 to match
Parts:
- removed R166, R172, R174, R176: 360mΩ ±5%, Resistor_SMD:R_0805_2012Metric, symbol JLCImport:RTT05R36JTP
- added R159, R160, R81, R82: 200mΩ ±1%, JLCImport:RL12FTNR200, symbol JLCImport:RL12FTNR200
Connections:
- net +12V: now also R159.1, R160.1, R81.1, R82.1
- net +12V_FAN0: now also R81.2
- net +12V_FAN1: now also R82.2
- net +12V_FAN2: now also R159.2
- net +12V_FAN3: now also R160.2
Other:
- note added: "~500mA rated sense for FAN0 on +12V"
- note added: "~500mA rated sense for FAN1 on +12V"
- note added: "~500mA rated sense for FAN2 on +12V"
- note added: "~500mA rated sense for FAN3 on +12V"
- note removed: "~275mA max sense for FAN0 on +12V"
- note removed: "~275mA max sense for FAN1 on +12V"
- note removed: "~275mA max sense for FAN2 on +12V"
- note removed: "~275mA max sense for FAN3 on +12V"
