File: pcb_files/PAC1954_PSU_PD.kicad_sch (KiCad schematic)
At the start: 10 parts, among them U24 PAC1954T-E_4MX

Commit message: Basic Function Review/Documentation for MCP9808
Parts:
- removed R146: 20mΩ ±1%, Resistor_SMD:R_0603_1608Metric, symbol JLCImport:RBL06FTR020
- removed R147, R148: 100k, Resistor_SMD:R_0402_1005Metric, symbol JLCImport:0402WGF1003TCE
- added R89, R90: 49.9k, Resistor_SMD:R_0402_1005Metric, symbol JLCImport:RMS04FT4992
Connections:
- net +3V3: now also R89.1, R90.2
- net SCL: now also R89.2
- net SDA: now also R90.1
- net VBUS: no longer names the net of U24.11 (SENSE1+)
- net VBUS_SENSE: no longer names the net of U24.12 (SENSE1-)
- no-connect marks 0 -> 2
Other:
- note removed: "~5 A max sense on USB-C VBUS"

Commit message: Switched PAC1954 to SLOW mode to save power
Parts:
- added C128: 100nF, Capacitor_SMD:C_0402_1005Metric, symbol JLCImport:CL05B104KB54PNC
- added C247: 4.7uF, Capacitor_SMD:C_0402_1005Metric, symbol JLCImport:CL05A475MP5NRNC
Connections:
- net +3V3: now also R144.2; no longer R141.2, R89.1, R90.2, U24.2 (VDD)
- net GND: now also C128.1, C247.1; no longer R144.2
- new net VDD: C128.2, C247.2, R141.2, R89.1, R90.2, U24.2 (VDD)
Other:
- note added: "Pull up to enable SLOW sampling"
- note removed: "Pull down to disable SLOW sampling"

Commit message: Added FAN4 and updated RP2354/PAC1954 to match
Parts:
- added R162: 200mΩ ±1%, JLCImport:RL12FTNR200, symbol JLCImport:RL12FTNR200
Connections:
- net +3V3 is gone; now on net VDD: R144.2, R145.2, U24.9 (SENSE4-)
- net +12V: now also U24.11 (SENSE1+), R162.1
- net +12V_FAN4: now reaches U24.12 (SENSE1-)
- net +12V_FAN4: now also R162.2
- no-connect marks 2 -> 0
Other:
- note added: "~500mA rated sense for FAN4 on +12V"
Changed lines of the file:
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@@
+		)
+	)
+	(text "~500mA rated sense for FAN4 on +12V"
+		(exclude_from_sim no)
+		(at 92.71 89.408 0)
+		(effects
+			(font
+				(size 0.9144 0.9144)
+			)
 		)
 	)
@@
 		(color 0 0 0 0)
 	)
-	(no_connect
-		(at 100.33 50.8)
-	)
-	(no_connect
-		(at 100.33 53.34)
-	)
 	(wire
 		(pts
@@
 	(wire
 		(pts
+			(xy 100.33 53.34) (xy 105.41 53.34)
+		)
+		(stroke
+			(width 0)
+			(type default)
+		)
+	)
+	(wire
+		(pts
 			(xy 125.73 76.2) (xy 133.35 76.2)
 		)
@@
 	(wire
 		(pts
+			(xy 83.82 86.36) (xy 87.63 86.36)
+		)
+		(stroke
+			(width 0)
+			(type default)
+		)
+	)
+	(wire
+		(pts
 			(xy 124.46 66.04) (xy 125.73 66.04)
 		)
@@
 	(wire
 		(pts
+			(xy 100.33 50.8) (xy 105.41 50.8)
+		)
+		(stroke
+			(width 0)
+			(type default)
+		)
+	)
+	(wire
+		(pts
 			(xy 102.87 36.83) (xy 105.41 36.83)
 		)
@@
 	(wire
 		(pts
+			(xy 100.33 86.36) (xy 97.79 86.36)
+		)
+		(stroke
+			(width 0)
+			(type default)
+		)
+	)
+	(wire
+		(pts
 			(xy 48.26 54.61) (xy 52.07 54.61)
 		)
@@
 		)
 	)
+	(hierarchical_label "VDD"
+		(shape input)
+		(at 48.26 57.15 180)
+		(effects
+			(font
+				(size 1.27 1.27)
+			)
+			(justify right)
+		)
+	)
 	(hierarchical_label "PSU_+5VDC"
 		(shape input)
@@
 		)
 	)
+	(hierarchical_label "+12V_FAN4"
+		(shape output)
+		(at 105.41 50.8 0)
+		(effects
+			(font
+				(size 1.27 1.27)
+			)
+			(justify left)
+		)
+	)
 	(hierarchical_label "PSU_+3V3DC"
 		(shape input)
@@
 		)
 	)
-	(hierarchical_label "+3V3"
+	(hierarchical_label "+12V"
+		(shape bidirectional)
+		(at 83.82 86.36 180)
+		(effects
+			(font
+				(size 1.27 1.27)
+			)
+			(justify right)
+		)
+	)
+	(hierarchical_label "VDD"
 		(shape input)
 		(at 63.5 26.67 0)
@@
 		)
 	)
-	(hierarchical_label "+3V3"
+	(hierarchical_label "VDD"
 		(shape input)
 		(at 66.04 86.36 0)
@@
 	)
 	(hierarchical_label "+12V"
-		(shape output)
+		(shape bidirectional)
 		(at 48.26 52.07 180)
 		(effects
@@
 		(shape input)
 		(at 48.26 41.91 180)
-		(effects
-			(font
-				(size 1.27 1.27)
-			)
-			(justify right)
-		)
-	)
-	(hierarchical_label "+3V3"
-		(shape input)
-		(at 48.26 57.15 180)
 		(effects
 			(font
@@
 		)
 	)
+	(hierarchical_label "+12V"
+		(shape bidirectional)
+		(at 105.41 53.34 0)
+		(effects
+			(font
+				(size 1.27 1.27)
+			)
+			(justify left)
+		)
+	)
 	(hierarchical_label "PSU_+3V3DC"
 		(shape input)
@@
 	)
 	(hierarchical_label "+12V"
+		(shape bidirectional)
+		(at 64.77 71.12 0)
+		(effects
+			(font
+				(size 1.27 1.27)
+			)
+			(justify left)
+		)
+	)
+	(hierarchical_label "+12V_FAN4"
 		(shape output)
-		(at 64.77 71.12 0)
+		(at 100.33 86.36 0)
 		(effects
 			(font
@@
 					(unit 1)
 				)
+			)
+		)
+	)
+	(symbol
+		(lib_id "JLCImport:RL12FTNR200")
+		(at 92.71 86.36 0)
+		(unit 1)
+		(body_style 1)
+		(exclude_from_sim no)
+		(in_bom yes)
+		(on_board yes)
+		(in_pos_files yes)
+		(dnp no)
+		(fields_autoplaced yes)
+		(property "Reference" "R162"
+			(at 92.71 80.01 0)
+			(show_name no)
+			(do_not_autoplace no)
+			(effects
+				(font
+					(size 1.27 1.27)
+				)
+			)
+		)
+		(property "Value" "200mΩ ±1%"
+			(at 92.71 82.55 0)
+			(show_name no)
+			(do_not_autoplace no)
+			(effects
+				(font
+					(size 1.27 1.27)
+				)
+			)
+		)
+		(property "Footprint" "JLCImport:RL12FTNR200"
+			(at 92.71 86.36 0)
+			(hide yes)
+			(show_name no)
+			(do_not_autoplace no)
+			(effects
+				(font
+					(size 1.27 1.27)
+				)
+			)
+		)
+		(property "Datasheet" "https://www.lcsc.com/datasheet/lcsc_datasheet_2304140030_TA-I-Tech-RL12FTNR200_C160920.pdf"
+			(at 92.71 86.36 0)
+			(hide yes)
+			(show_name no)
+			(do_not_autoplace no)
+			(effects
+				(font
+					(size 1.27 1.27)
+				)
+			)
+		)
+		(property "Description" "200mΩ 500mW Metal Film Resistor SMD ±1% ±200ppm/℃ 1206 Current Sense Resistors / Shunt Resistors ROHS"
+			(at 92.71 86.36 0)
+			(hide yes)
+			(show_name no)
+			(do_not_autoplace no)
+			(effects
+				(font
+					(size 1.27 1.27)
+				)
+			)
+		)
+		(property "LCSC" "C160920"
+			(at 92.71 86.36 0)
+			(hide yes)
+			(show_name no)
+			(do_not_autoplace no)
+			(effects
+				(font
+					(size 1.27 1.27)
+				)
+			)
+		)
+		(property "Manufacturer" "TA-I Tech"
+			(at 92.71 86.36 0)
+			(hide yes)
+			(show_name no)
+			(do_not_autoplace no)
+			(effects
+				(font
+					(size 1.27 1.27)
+				)
+			)
+		)
+		(property "Manufacturer Part" "RL12FTNR200"
+			(at 92.71 86.36 0)
+			(hide yes)
+			(show_name no)
+			(do_not_autoplace no)
+			(effects
+				(font
+					(size 1.27 1.27)
+				)
+			)
+		)
+		(pin "1"
+		)
+		(pin "2"
+		)
+		(instances
+			(project "serverv2_backplane"
+				(path "/d38d6818-cf53-410d-afa3-a75a85b7c05a/b93a12c2-f637-489d-8857-c7fe286f64a4"
+					(reference "R162")
+					(unit 1)
+				)

Commit message: Basic Function Review/Documentation for PSU PAC1954
Parts:
- removed R140: 3mΩ ±1%, Resistor_SMD:R_1206_3216Metric, symbol JLCImport:YHR1206SE1WR003F5
- removed R145: 14mΩ ±1%, Resistor_SMD:R_0805_2012Metric, symbol JLCImport:YHR1206SE1WR003F5
- added R166: 2.5mΩ ±1%, Resistor_SMD:R_2512_6332Metric, symbol JLCImport:JER2512F3R2R5L
- added R170: 68mΩ ±1%, Resistor_SMD:R_1206_3216Metric, symbol JLCImport:YHR1206SE1WR003F5
Connections:
- net +12V: now also R166.2
- net PSU_+12V1DC: now also R166.1
- net PSU_+3V3DC: now also R170.1
- net VDD: now also R170.2
Other:
- note added: "~1.47 A max sense on 3V3 rail"
- note added: "~40 A max sense on 12V rail"
- note removed: "~32 A max sense on 12V rail"
- note removed: "~7 A max sense on 3V3 rail"
Changed lines of the file:
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@@
 		)
 	)
-	(text "~32 A max sense on 12V rail"
+	(text "~40 A max sense on 12V rail"
 		(exclude_from_sim no)
 		(at 57.912 74.676 0)
@@
 		)
 	)
-	(text "~7 A max sense on 3V3 rail"
+	(text "~1.47 A max sense on 3V3 rail"
 		(exclude_from_sim no)
 		(at 58.42 90.424 0)
@@
 				(path "/d38d6818-cf53-410d-afa3-a75a85b7c05a/b93a12c2-f637-489d-8857-c7fe286f64a4"
 					(reference "C128")
-					(unit 1)
-				)
-			)
-		)
-	)
-	(symbol
-		(lib_id "JLCImport:YHR1206SE1WR003F5")
-		(at 58.42 86.36 0)
-		(unit 1)
-		(body_style 1)
-		(exclude_from_sim no)
-		(in_bom yes)
-		(on_board yes)
-		(in_pos_files yes)
-		(dnp no)
-		(property "Reference" "R145"
-			(at 58.42 81.026 0)
-			(show_name no)
-			(do_not_autoplace no)
-			(effects
-				(font
-					(size 1.27 1.27)
-				)
-			)
-		)
-		(property "Value" "14mΩ ±1%"
-			(at 58.42 83.566 0)
-			(show_name no)
-			(do_not_autoplace no)
-			(effects
-				(font
-					(size 1.27 1.27)
-				)
-			)
-		)
-		(property "Footprint" "Resistor_SMD:R_0805_2012Metric"
-			(at 58.42 86.36 0)
-			(hide yes)
-			(show_name no)
-			(do_not_autoplace no)
-			(effects
-				(font
-					(size 1.27 1.27)
-				)
-			)
-		)
-		(property "Datasheet" "https://www.lcsc.com/datasheet/C2941109.pdf?spm=wm.sxq.inf.ggs___wm.fly.bg.0.xh&lcsc_vid=FgcLV1deR1RZUAZfQwALU1UCEQMPU1IETwdYAQAFQAUxVlNeRFZdX11QRlhdVjsOAxUeFF5JWBYZEEoKFBINSQcJGk4NBhADEA4cHktXRlhXSQwSGg0%3D"
-			(at 58.42 86.36 0)
-			(hide yes)
-			(show_name no)
-			(do_not_autoplace no)
-			(effects
-				(font
-					(size 1.27 1.27)
-				)
-			)
-		)
-		(property "Description" "RES 14mΩ ±1% 500mW 0805"
-			(at 58.42 86.36 0)
-			(hide yes)
-			(show_name no)
-			(do_not_autoplace no)
-			(effects
-				(font
-					(size 1.27 1.27)
-				)
-			)
-		)
-		(property "LCSC" "C2941109"
-			(at 58.42 86.36 0)
-			(hide yes)
-			(show_name no)
-			(do_not_autoplace no)
-			(effects
-				(font
-					(size 1.27 1.27)
-				)
-			)
-		)
-		(property "Manufacturer" "UNI-ROYAL"
-			(at 58.42 86.36 0)
-			(hide yes)
-			(show_name no)
-			(do_not_autoplace no)
-			(effects
-				(font
-					(size 1.27 1.27)
-				)
-			)
-		)
-		(property "Manufacturer Part" "MS05W2F140MT5E"
-			(at 58.42 86.36 0)
-			(hide yes)
-			(show_name no)
-			(do_not_autoplace no)
-			(effects
-				(font
-					(size 1.27 1.27)
-				)
-			)
-		)
-		(pin "1"
-		)
-		(pin "2"
-		)
-		(instances
-			(project "serverv2_backplane"
-				(path "/d38d6818-cf53-410d-afa3-a75a85b7c05a/b93a12c2-f637-489d-8857-c7fe286f64a4"
-					(reference "R145")
 					(unit 1)
 				)
@@
 	(symbol
 		(lib_id "JLCImport:YHR1206SE1WR003F5")
+		(at 58.42 86.36 0)
+		(unit 1)
+		(body_style 1)
+		(exclude_from_sim no)
+		(in_bom yes)
+		(on_board yes)
+		(in_pos_files yes)
+		(dnp no)
+		(property "Reference" "R170"
+			(at 58.42 81.026 0)
+			(show_name no)
+			(do_not_autoplace no)
+			(effects
+				(font
+					(size 1.27 1.27)
+				)
+			)
+		)
+		(property "Value" "68mΩ ±1%"
+			(at 58.42 83.566 0)
+			(show_name no)
+			(do_not_autoplace no)
+			(effects
+				(font
+					(size 1.27 1.27)
+				)
+			)
+		)
+		(property "Footprint" "Resistor_SMD:R_1206_3216Metric"
+			(at 58.42 86.36 0)
+			(hide yes)
+			(show_name no)
+			(do_not_autoplace no)
+			(effects
+				(font
+					(size 1.27 1.27)
+				)
+			)
+		)
+		(property "Datasheet" "https://www.lcsc.com/datasheet/C2874764.pdf?spm=wm.sxq.inf.ggs___wm.fly.bg.9.xh&lcsc_vid=FgcLV1deR1RZUAZfQwALU1UCEQMPU1IETwdYAQAFQAUxVlNeRFZdX11QRlhdVjsOAxUeFF5JWBYZEEoKFBINSQcJGk4NBhADEA4cHktXRlhXSQwSGg0%3D"
+			(at 58.42 86.36 0)
+			(hide yes)
+			(show_name no)
+			(do_not_autoplace no)
+			(effects
+				(font
+					(size 1.27 1.27)
+				)
+			)
+		)
+		(property "Description" "RES 68mΩ ±1% 1W 1206"
+			(at 58.42 86.36 0)
+			(hide yes)
+			(show_name no)
+			(do_not_autoplace no)
+			(effects
+				(font
+					(size 1.27 1.27)
+				)
+			)
+		)
+		(property "LCSC" "C42454045"
+			(at 58.42 86.36 0)
+			(hide yes)
+			(show_name no)
+			(do_not_autoplace no)
+			(effects
+				(font
+					(size 1.27 1.27)
+				)
+			)
+		)
+		(property "Manufacturer" "Yohey"
+			(at 58.42 86.36 0)
+			(hide yes)
+			(show_name no)
+			(do_not_autoplace no)
+			(effects
+				(font
+					(size 1.27 1.27)
+				)
+			)
+		)
+		(property "Manufacturer Part" "YHR1206SE1WR068F5"
+			(at 58.42 86.36 0)
+			(hide yes)
+			(show_name no)
+			(do_not_autoplace no)
+			(effects
+				(font
+					(size 1.27 1.27)
+				)
+			)
+		)
+		(pin "1"
+		)
+		(pin "2"
+		)
+		(instances
+			(project "serverv2_backplane"
+				(path "/d38d6818-cf53-410d-afa3-a75a85b7c05a/b93a12c2-f637-489d-8857-c7fe286f64a4"
+					(reference "R170")
+					(unit 1)
+				)
+			)
+		)
+	)
+	(symbol
+		(lib_id "JLCImport:YHR1206SE1WR003F5")
 		(at 92.71 71.12 0)
 		(unit 1)
@@
 	)
 	(symbol
+		(lib_id "JLCImport:JER2512F3R2R5L")
+		(at 58.42 71.12 0)
+		(unit 1)
+		(body_style 1)
+		(exclude_from_sim no)
+		(in_bom yes)
+		(on_board yes)
+		(in_pos_files yes)
+		(dnp no)
+		(fields_autoplaced yes)
+		(property "Reference" "R166"
+			(at 58.42 64.77 0)
+			(show_name no)
+			(do_not_autoplace no)
+			(effects
+				(font
+					(size 1.27 1.27)
+				)
+			)
+		)
+		(property "Value" "2.5mΩ ±1%"
+			(at 58.42 67.31 0)
+			(show_name no)
+			(do_not_autoplace no)
+			(effects
+				(font
+					(size 1.27 1.27)
+				)
+			)
+		)
+		(property "Footprint" "Resistor_SMD:R_2512_6332Metric"
+			(at 58.42 71.12 0)
+			(hide yes)
+			(show_name no)
+			(do_not_autoplace no)
+			(effects
+				(font
+					(size 1.27 1.27)
+				)
+			)
+		)
+		(property "Datasheet" "https://www.lcsc.com/datasheet/lcsc_datasheet_2506121200_jieerrui-JER2512F3R2R5L_C49164684.pdf"
+			(at 58.42 71.12 0)
+			(hide yes)
+			(show_name no)
+			(do_not_autoplace no)
+			(effects
+				(font
+					(size 1.27 1.27)
+				)
+			)
+		)
+		(property "Description" "2.5mΩ 3W Current Sense Resistor SMD ±1% ±50ppm/℃ 2512 Current Sense Resistors / Shunt Resistors ROHS"
+			(at 58.42 71.12 0)
+			(hide yes)
+			(show_name no)
+			(do_not_autoplace no)
+			(effects
+				(font
+					(size 1.27 1.27)
+				)
+			)
+		)
+		(property "LCSC" "C49164684"
+			(at 58.42 71.12 0)
+			(hide yes)
+			(show_name no)
+			(do_not_autoplace no)
+			(effects
+				(font
+					(size 1.27 1.27)
+				)
+			)
+		)
+		(property "Manufacturer" "jieerrui"
+			(at 58.42 71.12 0)
+			(hide yes)
+			(show_name no)
+			(do_not_autoplace no)
+			(effects
+				(font
+					(size 1.27 1.27)
+				)
+			)
+		)
+		(property "Manufacturer Part" "JER2512F3R2R5L"
+			(at 58.42 71.12 0)
+			(hide yes)
+			(show_name no)
+			(do_not_autoplace no)
+			(effects
+				(font
+					(size 1.27 1.27)
+				)
+			)
+		)
+		(pin "1"
+		)
+		(pin "2"
+		)
+		(instances
+			(project "serverv2_backplane"
+				(path "/d38d6818-cf53-410d-afa3-a75a85b7c05a/b93a12c2-f637-489d-8857-c7fe286f64a4"
+					(reference "R166")
+					(unit 1)
+				)
+			)
+		)
+	)
+	(symbol
 		(lib_id "JLCImport:CL05A475MP5NRNC")
 		(at 133.35 71.12 90)
@@
 					(unit 1)
 				)
-			)
-		)
-	)
-	(symbol
-		(lib_id "JLCImport:YHR1206SE1WR003F5")
-		(at 58.42 71.12 0)
-		(unit 1)
-		(body_style 1)
-		(exclude_from_sim no)
-		(in_bom yes)
-		(on_board yes)
-		(in_pos_files yes)
-		(dnp no)
-		(property "Reference" "R140"
-			(at 58.42 65.786 0)
-			(show_name no)
-			(do_not_autoplace no)
-			(effects
-				(font
-					(size 1.27 1.27)
-				)
-			)
-		)
-		(property "Value" "3mΩ ±1%"
-			(at 58.42 68.326 0)
-			(show_name no)
-			(do_not_autoplace no)
-			(effects
-				(font
-					(size 1.27 1.27)
-				)
-			)
-		)
-		(property "Footprint" "Resistor_SMD:R_1206_3216Metric"
-			(at 58.42 71.12 0)
-			(hide yes)
-			(show_name no)
-			(do_not_autoplace no)
-			(effects
-				(font
-					(size 1.27 1.27)
-				)
-			)
-		)
-		(property "Datasheet" "https://atta.szlcsc.com/upload/public/pdf/source/20250120/0C9113E53EE977994BFB208E06A9E207.pdf"
-			(at 58.42 71.12 0)
-			(hide yes)
-			(show_name no)
-			(do_not_autoplace no)
-			(effects
-				(font
-					(size 1.27 1.27)
-				)
-			)
-		)
-		(property "Description" "3mΩ ±1% 1W 温度系数：50PPM"
-			(at 58.42 71.12 0)
-			(hide yes)
-			(show_name no)
-			(do_not_autoplace no)
-			(effects
-				(font
-					(size 1.27 1.27)
-				)
-			)
-		)
-		(property "LCSC" "C42454016"
-			(at 58.42 71.12 0)
-			(hide yes)
-			(show_name no)
-			(do_not_autoplace no)
-			(effects
-				(font
-					(size 1.27 1.27)
-				)
-			)
-		)
-		(property "Manufacturer" "Yohey(元晖)"
-			(at 58.42 71.12 0)
-			(hide yes)
-			(show_name no)
-			(do_not_autoplace no)
-			(effects
-				(font
-					(size 1.27 1.27)
-				)
-			)
-		)
-		(property "Manufacturer Part" "YHR1206SE1WR003F5"
-			(at 58.42 71.12 0)
-			(hide yes)
-			(show_name no)
-			(do_not_autoplace no)
-			(effects
-				(font
-					(size 1.27 1.27)
-				)
-			)
-		)
-		(pin "1"
-		)
-		(pin "2"
-		)
-		(instances
-			(project "serverv2_backplane"
-				(path "/d38d6818-cf53-410d-afa3-a75a85b7c05a/b93a12c2-f637-489d-8857-c7fe286f64a4"
-					(reference "R140")
-					(unit 1)
-				)
